File: mecc-pcb-kicad.kicad_pcb (KiCad board)
At the start: 2 copper layers, 230.1 x 130 mm, 67 parts, among them J1 VESC Term, J2 STM SIGS, J4 4.9V, J5 PDQE15-Q48-D24-D, Q1 NMOS, Q2 NMOS, Q3 PMOS, Q4 PMOS, U1 SEN-16407, U2 SN74HCS09QPWRQ1, U3 SN74LVC1G139DCUR

Commit message: Fixing Becca's Comments 11-2-23
Parts:
- U1: Current Sensor: renamed from U1
- moved DISCHARGE_RELAY1 33.7 mm to (197.3, 167.0)
- moved Q1 33.6 mm to (157.7, 187.1)
- moved Q3 33.6 mm to (163.9, 165.8)
- moved RHIGH_10k2 33.6 mm to (166.6, 194.2)
- moved RHIGH_10k3 33.6 mm to (166.6, 179.1)
- moved RHIGH_10k5 33.6 mm to (166.6, 172.0)
- moved TP2 33.6 mm to (150.2, 179.1)
- moved TP3 33.6 mm to (166.9, 187.8)
- moved D4 33.6 mm to (173.3, 175.2)
- moved R_RELAY_PULLDOWN4 33.6 mm to (174.0, 183.5)
- moved U1: Current Sensor 14.5 mm to (251.7, 151.6)
Routing:
- net +5V: track 212.1 -> 179.0 mm, vias 0 -> 5
- net PRE_LOW_DIS: track 195.5 -> 227.0 mm
- net GND: track 835.5 -> 809.4 mm
- net VESC_NEG: track 170.3 -> 190.8 mm
- net VESC_POS: track 76.7 -> 89.8 mm
- net Net-(HIGH_SIDE_RELAY1-NO): track 36.8 -> 24.9 mm
- net BATT_V_SENSOR: track 328.0 -> 316.2 mm, vias 3 -> 5
- net BATT_CURR_SENSOR: track 261.3 -> 272.0 mm, vias 2 -> 1
- net Net-(Q3-G): track 24.4 -> 34.5 mm
- net Net-(DISCHARGE_RELAY1-NC): track 31.4 -> 39.8 mm
- net PRE_LOW_DIS_STM: track 129.8 -> 137.1 mm
Other:
- board text added: "WEC-PROTOTYPE PCB MK2 FA'23 Kelvin Resch (kr562) Nathan Rakhlin (npr29) Sabian Grier (srg293)"
- board text removed: "Contact us at no83@cornell.edu or am2389@cornell.edu."
- board text removed: "MECC v2"
- board text removed: "WEC-PROTOTYPE PCB MK2 FA'23 Kelvin Resch (kr562) Nathan Rakhlin (npr29)"

Commit message: Becca's messages
Parts:
- moved C2 20.7 mm to (131.2, 169.0)
- moved Torq Sensor 19.8 mm to (98.0, 168.4)
- moved R2 18.0 mm to (102.2, 152.6)
- moved R1 18.0 mm to (97.8, 160.2)
- moved J2 1.46 mm to (175.3, 137.0)
Routing:
- net GND: track 809.4 -> 831.4 mm
- net Net-(R1-Pad2): track 7.62 -> 26.2 mm
- net +24V: track 44.6 -> 63.0 mm
- net +5V: track 179.0 -> 188.5 mm
- net WAVE_GAUGE: track 35.7 -> 32.6 mm, vias 0 -> 1
- net TORQUE_SENSOR: track 7.40 -> 9.34 mm
- net HIGH_SIDE_STM: track 122.2 -> 121.6 mm
- net PRE_LOW_DIS_STM: track 137.1 -> 136.5 mm
